Commit message: Task E complete

File: body.urdf (robot description, URDF)
Before this commit: robot robot, 2 links, 1 joints
Links:
- removed link Leg
- added link BackLeg, mass 1; collision box size=1 1 1; visual box size=1 1 1
- added link FrontLeg, mass 1; collision box size=1 1 1; visual box size=1 1 1
Joints:
- removed joint Torso_Leg
- added joint Torso_BackLeg: type revolute, parent Torso, child BackLeg, origin xyz=1 0 1 rpy=0 0 0, axis 0 1 0, limit lower=-3.14159 upper=3.14159 effort=0.0 velocity=0.0
- added joint Torso_FrontLeg: type revolute, parent Torso, child FrontLeg, origin xyz=2.5 0 1 rpy=0 0 0, axis 0 1 0, limit lower=-3.14159 upper=3.14159 effort=0.0 velocity=0.0

Commit message: Fixed positions

File: body.urdf (robot description, URDF)
Before this commit: robot robot, 3 links, 2 joints
Joints:
- joint Torso_FrontLeg: origin xyz=2.5 0 1 rpy=0 0 0 -> xyz=2 0 1 rpy=0 0 0

Commit message: Robot body and environment done, think training might work testing rn

File: body.urdf (robot description, URDF)
Before this commit: robot robot, 3 links, 2 joints
Links:
- removed link BackLeg
- removed link FrontLeg
- added link LeftFoot, mass 1; collision box size=0.5 0.6 0.5; visual box size=0.5 0.6 0.5
- added link LeftLeg, mass 1; collision box size=0.5 0.3 1; visual box size=0.5 0.3 1
- added link LeftLegLower, mass 1; collision box size=0.5 0.3 1; visual box size=0.5 0.3 1
- added link RightFoot, mass 1; collision box size=0.5 0.6 0.5; visual box size=0.5 0.6 0.5
- added link RightLeg, mass 1; collision box size=0.5 0.3 1; visual box size=0.5 0.3 1
- added link RightLegLower, mass 1; collision box size=0.5 0.3 1; visual box size=0.5 0.3 1
- link Torso: geometry collision box size=0.5 2 2; visual box size=0.5 2 2
Joints:
- removed joint Torso_BackLeg
- removed joint Torso_FrontLeg
- added joint LeftLegLower_LeftFoot: type revolute, parent LeftLegLower, child LeftFoot, origin xyz=0 0 -1 rpy=0 0 0, axis 0 1 0, limit lower=-3.14159 upper=3.14159 effort=0.0 velocity=0.0
- added joint LeftLeg_LeftLegLower: type revolute, parent LeftLeg, child LeftLegLower, origin xyz=0 0 -1 rpy=0 0 0, axis 0 1 0, limit lower=-3.14159 upper=3.14159 effort=0.0 velocity=0.0
- added joint RightLegLower_RightFoot: type revolute, parent RightLegLower, child RightFoot, origin xyz=0 0 -1 rpy=0 0 0, axis 0 1 0, limit lower=-3.14159 upper=3.14159 effort=0.0 velocity=0.0
- added joint RightLeg_RightLegLower: type revolute, parent RightLeg, child RightLegLower, origin xyz=0 0 -1 rpy=0 0 0, axis 0 1 0, limit lower=-3.14159 upper=3.14159 effort=0.0 velocity=0.0
- added joint Torso_LeftLeg: type revolute, parent Torso, child LeftLeg, origin xyz=0 -1 2.5 rpy=0 0 0, axis 1 0 0, limit lower=-3.14159 upper=3.14159 effort=0.0 velocity=0.0
- added joint Torso_RightLeg: type revolute, parent Torso, child RightLeg, origin xyz=0 1 2.5 rpy=0 0 0, axis 1 0 0, limit lower=-3.14159 upper=3.14159 effort=0.0 velocity=0.0
